File: microcontroller.kicad_sch (KiCad schematic)
At the start: 20 parts, among them U4 RP2040, Y1 X322512MSB4SI

Commit message: design flaw fix
Parts:
- R10: value 1k -> DNF
Connections:
- net +1V1: no longer U4.44 (VREG_IN)
- net +3V3: now also U4.44 (VREG_IN)
Changed lines of the file:
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@@
   (junction (at 204.47 41.91) (diameter 0) (color 0 0 0 0)
   )
+  (junction (at 139.7 52.07) (diameter 0) (color 0 0 0 0)
+  )
   (junction (at 250.19 41.91) (diameter 0) (color 0 0 0 0)
   )
@@
   (junction (at 193.04 31.75) (diameter 0) (color 0 0 0 0)
   )
-  (junction (at 130.81 52.07) (diameter 0) (color 0 0 0 0)
-  )
   (wire (pts (xy 46.355 109.22) (xy 62.865 109.22))
     (stroke (width 0) (type default) (color 0 0 0 0))
@@
     (stroke (width 0) (type default) (color 0 0 0 0))
   )
-  (wire (pts (xy 134.62 52.07) (xy 134.62 58.42))
-    (stroke (width 0) (type default) (color 0 0 0 0))
-  )
   (wire (pts (xy 191.135 147.32) (xy 175.26 147.32))
     (stroke (width 0) (type default) (color 0 0 0 0))
@@
     (stroke (width 0) (type default) (color 0 0 0 0))
   )
-  (wire (pts (xy 130.81 52.07) (xy 134.62 52.07))
-    (stroke (width 0) (type default) (color 0 0 0 0))
-  )
   (wire (pts (xy 57.15 89.535) (xy 46.355 89.535))
     (stroke (width 0) (type default) (color 0 0 0 0))
@@
     (stroke (width 0) (type default) (color 0 0 0 0))
   )
+  (wire (pts (xy 139.7 52.07) (xy 142.24 52.07))
+    (stroke (width 0) (type default) (color 0 0 0 0))
+  )
   (wire (pts (xy 26.035 180.34) (xy 28.575 180.34))
     (stroke (width 0) (type default) (color 0 0 0 0))
@@
     (stroke (width 0) (type default) (color 0 0 0 0))
   )
+  (wire (pts (xy 134.62 58.42) (xy 134.62 52.07))
+    (stroke (width 0) (type default) (color 0 0 0 0))
+  )
   (polyline (pts (xy 15.24 25.4) (xy 41.275 25.4))
     (stroke (width 0) (type default) (color 0 0 0 0))
@@
     (stroke (width 0) (type default) (color 0 0 0 0))
   )
-  (wire (pts (xy 139.7 52.07) (xy 142.24 52.07))
+  (wire (pts (xy 134.62 52.07) (xy 139.7 52.07))
     (stroke (width 0) (type default) (color 0 0 0 0))
   )
@@
     (in_bom yes) (on_board yes)
     (property "Reference" "R10" (id 0) (at 62.865 182.88 90))
-    (property "Value" "1k" (id 1) (at 62.865 177.8 90))
+    (property "Value" "DNF" (id 1) (at 62.865 177.8 90))
     (property "Footprint" "Resistor_SMD:R_0402_1005Metric" (id 2) (at 62.865 182.118 90)
       (effects (font (size 1.27 1.27)) hide)

Commit message: Remove trace under usb trace
Parts:
- R10: value DNF -> 100
Changed lines of the file:
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@@
   (symbol (lib_id "Device:R") (at 62.865 180.34 90) (unit 1)
     (in_bom yes) (on_board yes)
-    (property "Reference" "R10" (id 0) (at 62.865 182.88 90))
-    (property "Value" "DNF" (id 1) (at 62.865 177.8 90))
+    (property "Reference" "R10" (id 0) (at 62.865 178.181 90))
+    (property "Value" "100" (id 1) (at 62.865 182.88 90))
     (property "Footprint" "Resistor_SMD:R_0402_1005Metric" (id 2) (at 62.865 182.118 90)
       (effects (font (size 1.27 1.27)) hide)
