File: connectors.kicad_sch (KiCad schematic)
At the start: 5 parts, among them J1 Conn_02x05_Odd_Even, J2 USB_C_Receptacle_USB2.0, J3 Conn_02x21_Odd_Even

Commit message: design flaw fix
Connections:
- net USB_D+: no longer J3.35 (Pin_35), J3.36 (Pin_36)
- net USB_D-: no longer J3.37 (Pin_37), J3.38 (Pin_38)
- no-connect marks 5 -> 9
Changed lines of the file:
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@@
   (no_connect (at 48.895 171.45))
   (no_connect (at 48.895 168.91))
+  (no_connect (at 41.91 124.46))
+  (no_connect (at 54.61 124.46))
+  (no_connect (at 54.61 121.92))
   (no_connect (at 116.84 177.8))
+  (no_connect (at 41.91 121.92))
   (polyline (pts (xy 14.605 144.145) (xy 81.28 144.145))
     (stroke (width 0) (type default) (color 0 0 0 0))
@@
     (stroke (width 0) (type default) (color 0 0 0 0))
   )
-  (wire (pts (xy 24.13 124.46) (xy 41.91 124.46))
-    (stroke (width 0) (type default) (color 0 0 0 0))
-  )
   (wire (pts (xy 103.505 147.32) (xy 112.395 147.32))
     (stroke (width 0) (type default) (color 0 0 0 0))
@@
     (stroke (width 0) (type default) (color 0 0 0 0))
   )
-  (wire (pts (xy 72.39 121.92) (xy 54.61 121.92))
-    (stroke (width 0) (type default) (color 0 0 0 0))
-  )
   (wire (pts (xy 57.15 119.38) (xy 57.15 93.98))
     (stroke (width 0) (type default) (color 0 0 0 0))
@@
     (stroke (width 0) (type default) (color 0 0 0 0))
   )
-  (wire (pts (xy 24.13 121.92) (xy 41.91 121.92))
-    (stroke (width 0) (type default) (color 0 0 0 0))
-  )
   (wire (pts (xy 33.02 166.37) (xy 33.02 168.91))
     (stroke (width 0) (type default) (color 0 0 0 0))
@@
   )
   (wire (pts (xy 103.505 145.415) (xy 103.505 147.32))
-    (stroke (width 0) (type default) (color 0 0 0 0))
-  )
-  (wire (pts (xy 72.39 124.46) (xy 54.61 124.46))
     (stroke (width 0) (type default) (color 0 0 0 0))
   )
@@
     (effects (font (size 1.27 1.27)) (justify right bottom))
   )
-  (label "USB_D-" (at 24.13 124.46 0)
-    (effects (font (size 1.27 1.27)) (justify left bottom))
-  )
   (label "USER_IO_0" (at 72.39 81.28 180)
     (effects (font (size 1.27 1.27)) (justify right bottom))
@@
     (effects (font (size 1.27 1.27)) (justify right bottom))
   )
-  (label "USB_D-" (at 72.39 124.46 180)
-    (effects (font (size 1.27 1.27)) (justify right bottom))
-  )
   (label "USER_IO_2" (at 72.39 86.36 180)
     (effects (font (size 1.27 1.27)) (justify right bottom))
@@
     (effects (font (size 1.27 1.27)) (justify right bottom))
   )
-  (label "USB_D+" (at 24.13 121.92 0)
-    (effects (font (size 1.27 1.27)) (justify left bottom))
-  )
   (label "USER_IO_1" (at 24.13 83.82 0)
     (effects (font (size 1.27 1.27)) (justify left bottom))
@@
     (effects (font (size 1.27 1.27)) (justify right bottom))
   )
-  (label "USB_D+" (at 72.39 121.92 180)
-    (effects (font (size 1.27 1.27)) (justify right bottom))
-  )
